Commit message: Final environment class and test scripts before the test (#43)
* new user branch

* Resolve formatting issues on test scripts

* Resolve formatting issues on test scripts

File: urdf/block/model.urdf (robot description, URDF)
Before this commit: robot block, 1 links, 0 joints
Links:
- link block: geometry collision box size=0.0001 0.0001 0.0001; visual box size=0.05 0.05 0.05
